File: KiCad/PCI_Blaster/PCI_Blaster.kicad_sch (KiCad schematic)
At the start: 10 parts, among them J1 Bus_PCI_32bit_5V, U1 AMS1117CD-3.3

Commit message: redo pcb layout
Parts:
- removed D2: 1N4005, Diode_THT:D_DO-41_SOD81_P7.62mm_Horizontal, symbol Device:D
- removed TP1: +3.3V, Connector_PinSocket_2.54mm:PinSocket_1x01_P2.54mm_Vertical, symbol Connector:TestPoint
- removed TP2: GND, Connector_PinSocket_2.54mm:PinSocket_1x01_P2.54mm_Vertical, symbol Connector:TestPoint
- added JP1: Output Enable, Connector_PinHeader_2.54mm:PinHeader_1x02_P2.54mm_Vertical, symbol Jumper:Jumper_2_Bridged
- D1: value 1N4005 -> SB140
- LED1: value +3,3V -> +3.3V; footprint LED_THT:LED_D5.0mm -> LED_THT:LED_D3.0mm
- R1: footprint Resistor_THT:R_Axial_DIN0207_L6.3mm_D2.5mm_P10.16mm_Horizontal -> Resistor_THT:R_Axial_DIN0204_L3.6mm_D1.6mm_P5.08mm_Horizontal
- U1: footprint Package_TO_SOT_SMD:TO-252-3_TabPin2 -> Package_TO_SOT_SMD:TO-252-2
Connections:
- net +3.3V: now also JP1.2 (B); no longer C2.1, D1.2 (A), U1.2 (VO)
- net +5V: no longer J1.A10 (+5V), J1.A16 (+5V), J1.A59 (+5V), J1.B19 (+5V), J1.B59 (+5V)
- net GND: now also J1.A42 (GND); no longer J1.A12 (GND), J1.A13 (GND), J1.B12 (GND), J1.B13 (GND), J1.B17 (GND), J1.B46 (GND)
- new net V_OUT: C2.1, D1.2 (A), JP1.1 (A), U1.2 (VO)
- no-connect marks 0 -> 84
Other:
- company: (none) -> Undefined Systems, LLC
- title: (none) -> PCI Blaster
